Commit message: update launch code

File: src/robots/m1_description/urdf/xyuan_description_right_link.urdf (robot description, URDF)
Before this commit: robot xyuan_description, 29 links, 28 joints
Links:
- removed link dummy_link
- added link world
Joints:
- joint dummy_to_base_link: parent dummy_link -> world
